File: Prueba-01/encoderFilter/untitled.brd (EAGLE design)
At the start: 23.4 x 48.6 mm, 15 parts, among them Q1 IRF540, Q2 IRF540, Q3 IRF540

Commit message: update brd
Parts:
- added JP4: (no value), pinhead:1X02
Connections:
- net GND: now also JP4.2
- net VCC: now also JP4.1
Routing:
- net VCC: track 18.3 -> 29.7 mm
- net GND: track 97.0 -> 100.0 mm
- net N$1: track 53.5 -> 55.7 mm
Changed lines of the file:
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@@
 <attribute name="VALUE" x="18.88" y="7.255" size="1.27" layer="27" rot="R180"/>
+</element>
+<element name="JP4" library="pinhead" library_urn="urn:adsk.eagle:library:325" package="1X02" package3d_urn="urn:adsk.eagle:package:22435/2" value="" x="9.99" y="14.31" smashed="yes" rot="R90">
+<attribute name="5V" value="" x="9.99" y="14.31" size="1.778" layer="27" rot="R90" display="off"/>
+<attribute name="NAME" x="7.3512" y="12.5038" size="1.27" layer="25" ratio="10" rot="R90"/>
+<attribute name="POPULARITY" value="98" x="9.99" y="14.31" size="1.778" layer="27" rot="R90" display="off"/>
+<attribute name="VALUE" x="13.165" y="11.77" size="1.27" layer="27" rot="R90"/>
 </element>
 </elements>
@@
 <wire x1="20.25" y1="11.34" x2="20.25" y2="23.76" width="0.8128" layer="16"/>
 <wire x1="20.25" y1="23.76" x2="18.34" y2="25.67" width="0.8128" layer="16"/>
+<contactref element="JP4" pad="2"/>
+<wire x1="9.99" y1="15.58" x2="8.79" y2="16.78" width="0.8128" layer="1"/>
+<wire x1="8.79" y1="16.78" x2="7.45" y2="16.78" width="0.8128" layer="1"/>
 </signal>
 <signal name="N$1">
@@
 <wire x1="17.82" y1="42.39" x2="17.61" y2="42.18" width="0.8128" layer="16"/>
 <wire x1="20.52" y1="36.99" x2="20.52" y2="41.31" width="0.8128" layer="16"/>
-<wire x1="12.53" y1="22.57" x2="10.26" y2="24.84" width="0.8128" layer="16"/>
-<wire x1="10.26" y1="24.84" x2="10.26" y2="29.43" width="0.8128" layer="16"/>
-<wire x1="10.26" y1="29.43" x2="10.8" y2="29.97" width="0.8128" layer="16"/>
+<wire x1="10.8" y1="29.97" x2="10.26" y2="29.43" width="0.8128" layer="16"/>
 <wire x1="10.8" y1="35.1" x2="14.04" y2="38.34" width="0.8128" layer="16"/>
 <wire x1="14.04" y1="38.34" x2="15.66" y2="38.34" width="0.8128" layer="16"/>
 <wire x1="17.37" y1="36.63" x2="17.37" y2="35.91" width="0.8128" layer="16"/>
-<wire x1="12.53" y1="4.08" x2="12.53" y2="22.57" width="0.8128" layer="16"/>
 <wire x1="10.8" y1="29.97" x2="10.8" y2="35.1" width="0.8128" layer="16"/>
 <wire x1="15.66" y1="38.34" x2="17.37" y2="36.63" width="0.8128" layer="16"/>
+<wire x1="12.53" y1="6.64" x2="12.53" y2="4.08" width="0.8128" layer="16"/>
+<wire x1="10.26" y1="29.43" x2="10.26" y2="21.06" width="0.8128" layer="16"/>
+<wire x1="10.26" y1="21.06" x2="7.56" y2="18.36" width="0.8128" layer="16"/>
+<wire x1="7.56" y1="18.36" x2="7.56" y2="11.61" width="0.8128" layer="16"/>
+<wire x1="7.56" y1="11.61" x2="12.53" y2="6.64" width="0.8128" layer="16"/>
 </signal>
 <signal name="N$2">
@@
 <wire x1="16.66" y1="20.59" x2="12.39" y2="24.86" width="0.8128" layer="16"/>
 <wire x1="12.39" y1="24.86" x2="12.39" y2="26.94" width="0.8128" layer="16"/>
+<contactref element="JP4" pad="1"/>
+<wire x1="9.99" y1="13.04" x2="11.42" y2="13.04" width="0.8128" layer="16"/>
+<wire x1="13.23" y1="14.85" x2="13.23" y2="17.55" width="0.8128" layer="16"/>
+<wire x1="13.23" y1="17.55" x2="15.66" y2="19.98" width="0.8128" layer="16"/>
+<wire x1="15.66" y1="19.98" x2="16.2" y2="19.98" width="0.8128" layer="16"/>
+<wire x1="16.2" y1="19.98" x2="16.66" y2="20.44" width="0.8128" layer="16"/>
+<wire x1="16.66" y1="20.44" x2="16.66" y2="20.59" width="0.8128" layer="16"/>
+<wire x1="11.42" y1="13.04" x2="13.23" y2="14.85" width="0.8128" layer="16"/>
 </signal>
 </signals>
